Commit message: Working on urdf

File: fennee_description/urdf/fennee.xacro (robot description, xacro)
@@ -1,6 +1,6 @@
 <?xml version="1.0" encoding="UTF-8"?>
-<robot xmlns:xacro="http://www.ros.org/wiki/xacro" name="fenneeAI">
-   <material name="yellow">
-      <color rgba="0.92 0.83 0.0 1" />
+<robot xmlns:xacro="http://www.ros.org/wiki/xacro" name="fennee">
+   <material name="tan">
+      <color rgba="0.63 0.59 0.46 1" />
    </material>
    <material name="black">
@@ -11,5 +11,5 @@
    </material>
    <!-- Params -->
-   <xacro:property name="body_length" value="0.140" />
+   <xacro:property name="body_length" value="0.165" />
    <xacro:property name="body_width" value="0.110" />
    <xacro:property name="body_height" value="0.070" />
@@ -28,5 +28,6 @@
    <xacro:property name="shift" value="0.055" />
    <xacro:property name="shiftx" value="0.093" />
-   <xacro:property name="shifty" value="0.0395" />
+   <!-- <xacro:property name="shifty" value="0.0395" /> -->
+   <xacro:property name="shifty" value="0.04285" />
    <!-- Macros -->
    <xacro:macro name="gen_shoulder" params="name left">
@@ -94,5 +95,5 @@
                <origin rpy="0 0 3.1416" xyz="0.134 0.149 -0.0095" />
             </xacro:unless>
-            <material name="yellow" />
+            <material name="tan" />
          </visual>
       </link>
@@ -125,5 +126,5 @@
       </link>
       <gazebo reference="${name}_cover">
-         <material>Gazebo/ZincYellow</material>
+         <material>Gazebo/Grey</material>
       </gazebo>
    </xacro:macro>
@@ -272,5 +273,5 @@
          </geometry>
          <origin rpy="0 0 3.1416" xyz="0.042 0.055 -0.0195" />
-         <material name="yellow" />
+         <material name="tan" />
       </visual>
       <collision>
@@ -298,5 +299,5 @@
          </geometry>
          <origin rpy="0 0 3.1416" xyz="0.042 0.055 -0.0205" />
-         <material name="yellow" />
+         <material name="tan" />
       </visual>
       <collision>

File: fennee_description/urdf/stairs.urdf.xacro (robot description, xacro)
@@ -1,4 +1,4 @@
 <?xml version="1.0"?>
-<robot xmlns:xacro="http://www.ros.org/wiki/xacro" name="fenneeAI">
+<robot xmlns:xacro="http://www.ros.org/wiki/xacro" name="fennee">
     <material name="yellow">
         <color rgba="0.92 0.83 0.0 1"/>
