Commit message: Working on urdf

File: fennee_description/urdf/fennee.urdf (robot description, URDF)
Before this commit: robot fennee, 24 links, 23 joints
Links:
- link base_inertia: geometry collision box size=0.165 0.11 0.07; visual mesh filename=package://fennee_description/meshes/stl/mainbody.stl scale=0.001 0.001 0.001
Joints:
- joint front_left_shoulder: origin xyz=0.093 0.0395 0 rpy=0 0 0 -> xyz=0.093 0.04285 0 rpy=0 0 0
- joint front_right_shoulder: origin xyz=0.093 -0.0395 0 rpy=0 0 0 -> xyz=0.093 -0.04285 0 rpy=0 0 0
- joint rear_left_shoulder: origin xyz=-0.093 0.0395 0 rpy=0 0 0 -> xyz=-0.093 0.04285 0 rpy=0 0 0
- joint rear_right_shoulder: origin xyz=-0.093 -0.0395 0 rpy=0 0 0 -> xyz=-0.093 -0.04285 0 rpy=0 0 0

Commit message: Added oak d lite camera to urdf

File: fennee_description/urdf/fennee.urdf (robot description, URDF)
Before this commit: robot fennee, 24 links, 23 joints
Links:
- added link camera_left_camera_frame
- added link camera_left_camera_optical_frame
- added link camera_model_origin; visual mesh filename=package://depthai_descriptions/urdf/models/OAK-D-LITE.stl
- added link camera_rgb_camera_frame
- added link camera_rgb_camera_optical_frame
- added link camera_right_camera_frame
- added link camera_right_camera_optical_frame
- added link oak-d_frame
Joints:
- added joint camera_center_joint: type fixed, parent base_link, child oak-d_frame, origin xyz=0.169 0.0 -0.004 rpy=0.0 -0.174533 0.0
- added joint camera_left_camera_joint: type fixed, parent oak-d_frame, child camera_left_camera_frame, origin xyz=0 0.0375 0 rpy=0 0 0
- added joint camera_left_camera_optical_joint: type fixed, parent camera_left_camera_frame, child camera_left_camera_optical_frame, origin xyz=0 0 0 rpy=-1.5707963267948966 0.0 -1.5707963267948966
- added joint camera_model_origin_joint: type fixed, parent oak-d_frame, child camera_model_origin, origin xyz=0 0 0 rpy=1.5708 0 1.5708
- added joint camera_rgb_camera_joint: type fixed, parent oak-d_frame, child camera_rgb_camera_frame, origin xyz=0 0 0 rpy=0 0 0
- added joint camera_rgb_camera_optical_joint: type fixed, parent camera_rgb_camera_frame, child camera_rgb_camera_optical_frame, origin xyz=0 0 0 rpy=-1.5707963267948966 0.0 -1.5707963267948966
- added joint camera_right_camera_joint: type fixed, parent oak-d_frame, child camera_right_camera_frame, origin xyz=0 -0.0375 0 rpy=0 0 0
- added joint camera_right_camera_optical_joint: type fixed, parent camera_right_camera_frame, child camera_right_camera_optical_frame, origin xyz=0 0 0 rpy=-1.5707963267948966 0.0 -1.5707963267948966

File: fennee_description/urdf/fennee.xacro (robot description, xacro)
@@ -36,5 +36,6 @@
             <xacro:if value="${left}">
                <geometry>
-                  <mesh filename="package://fennee_description/meshes/stl/lshoulder.stl" scale="0.001 0.001 0.001" />
+                  <mesh filename="package://fennee_description/meshes/stl/lshoulder.stl"
+                     scale="0.001 0.001 0.001" />
                </geometry>
                <origin rpy="0 0 3.1416" xyz="0.135 0.0163 -0.0195" />
@@ -42,5 +43,6 @@
             <xacro:unless value="${left}">
                <geometry>
-                  <mesh filename="package://fennee_description/meshes/stl/rshoulder.stl" scale="0.001 0.001 0.001" />
+                  <mesh filename="package://fennee_description/meshes/stl/rshoulder.stl"
+                     scale="0.001 0.001 0.001" />
                </geometry>
                <origin rpy="0 0 3.1416" xyz="0.135 0.0938 -0.0205" />
@@ -66,5 +68,5 @@
          <axis xyz="1 0 0" />
          <origin rpy="0 0 0" xyz="${shiftx} ${shifty} 0" />
-         <limit effort="1000.0" velocity="0.7" lower="-0.548" upper="0.548"/>
+         <limit effort="1000.0" velocity="0.7" lower="-0.548" upper="0.548" />
          <dynamics damping="0.0" friction="0.5" />
       </joint>
@@ -72,9 +74,9 @@
          <type>transmission_interface/SimpleTransmission</type>
          <joint name="${pos}_shoulder">
-               <hardwareInterface>hardware_interface/PositionJointInterface</hardwareInterface>
+            <hardwareInterface>hardware_interface/PositionJointInterface</hardwareInterface>
          </joint>
          <actuator name="${pos}_shoulder_actuator">
-               <hardwareInterface>hardware_interface/PositionJointInterface</hardwareInterface>
-               <mechanicalReduction>1</mechanicalReduction>
+            <hardwareInterface>hardware_interface/PositionJointInterface</hardwareInterface>
+            <mechanicalReduction>1</mechanicalReduction>
          </actuator>
       </transmission>
@@ -85,5 +87,6 @@
             <xacro:if value="${left}">
                <geometry>
-                  <mesh filename="package://fennee_description/meshes/stl/larm_cover.stl" scale="0.001 0.001 0.001" />
+                  <mesh filename="package://fennee_description/meshes/stl/larm_cover.stl"
+                     scale="0.001 0.001 0.001" />
                </geometry>
                <origin rpy="0 0 3.1416" xyz="0.134 -0.04 -0.0095" />
@@ -91,5 +94,6 @@
             <xacro:unless value="${left}">
                <geometry>
-                  <mesh filename="package://fennee_description/meshes/stl/rarm_cover.stl" scale="0.001 0.001 0.001" />
+                  <mesh filename="package://fennee_description/meshes/stl/rarm_cover.stl"
+                     scale="0.001 0.001 0.001" />
                </geometry>
                <origin rpy="0 0 3.1416" xyz="0.134 0.149 -0.0095" />
@@ -102,5 +106,6 @@
             <xacro:if value="${left}">
                <geometry>
-                  <mesh filename="package://fennee_description/meshes/stl/larm.stl" scale="0.001 0.001 0.001" />
+                  <mesh filename="package://fennee_description/meshes/stl/larm.stl"
+                     scale="0.001 0.001 0.001" />
                </geometry>
                <origin rpy="0 0 3.1416" xyz="0.134 -0.04 -0.0095" />
@@ -108,5 +113,6 @@
             <xacro:unless value="${left}">
                <geometry>
-                  <mesh filename="package://fennee_description/meshes/stl/rarm.stl" scale="0.001 0.001 0.001" />
+                  <mesh filename="package://fennee_description/meshes/stl/rarm.stl"
+                     scale="0.001 0.001 0.001" />
                </geometry>
                <origin rpy="0 0 3.1416" xyz="0.134 0.149 -0.0095" />
@@ -135,5 +141,5 @@
          <axis xyz="0 1 0" />
          <origin rpy="0 0 0" xyz="0 ${shift} 0" />
-         <limit effort="1000.0" velocity="0.5" lower="-2.666" upper="1.548"/>
+         <limit effort="1000.0" velocity="0.5" lower="-2.666" upper="1.548" />
          <dynamics damping="0.0" friction="0.0" />
       </joint>
@@ -141,9 +147,9 @@
          <type>transmission_interface/SimpleTransmission</type>
          <joint name="${pos}_leg">
-               <hardwareInterface>hardware_interface/PositionJointInterface</hardwareInterface>
+            <hardwareInterface>hardware_interface/PositionJointInterface</hardwareInterface>
          </joint>
          <actuator name="${pos}_leg_actuator">
-               <hardwareInterface>hardware_interface/PositionJointInterface</hardwareInterface>
-               <mechanicalReduction>1</mechanicalReduction>
+            <hardwareInterface>hardware_interface/PositionJointInterface</hardwareInterface>
+            <mechanicalReduction>1</mechanicalReduction>
          </actuator>
       </transmission>
@@ -159,5 +165,6 @@
             <xacro:if value="${left}">
                <geometry>
-                  <mesh filename="package://fennee_description/meshes/stl/lfoot.stl" scale="0.001 0.001 0.001" />
+                  <mesh filename="package://fennee_description/meshes/stl/lfoot.stl"
+                     scale="0.001 0.001 0.001" />
                </geometry>
                <origin rpy="0 0 3.1416 " xyz="0.1195 -0.04 0.099" />
@@ -165,5 +172,6 @@
             <xacro:unless value="${left}">
                <geometry>
-                  <mesh filename="package://fennee_description/meshes/stl/rfoot.stl" scale="0.001 0.001 0.001" />
+                  <mesh filename="package://fennee_description/meshes/stl/rfoot.stl"
+                     scale="0.001 0.001 0.001" />
                </geometry>
                <origin rpy="0 0 3.1416" xyz="0.1195 0.149 0.099" />
@@ -189,5 +197,5 @@
          <axis xyz="0 1 0" />
          <origin rpy="0 0 0" xyz="0.014 0 -${leg_length}" />
-         <limit effort="1000.0" velocity="0.5" lower="-2.59" upper="0.1"/>
+         <limit effort="1000.0" velocity="0.5" lower="-2.59" upper="0.1" />
          <dynamics damping="0.0" friction="0.5" />
       </joint>
@@ -195,9 +203,9 @@
          <type>transmission_interface/SimpleTransmission</type>
          <joint name="${pos}_foot">
-               <hardwareInterface>hardware_interface/PositionJointInterface</hardwareInterface>
+            <hardwareInterface>hardware_interface/PositionJointInterface</hardwareInterface>
          </joint>
          <actuator name="${pos}_foot_actuator">
-               <hardwareInterface>hardware_interface/PositionJointInterface</hardwareInterface>
-               <mechanicalReduction>1</mechanicalReduction>
+            <hardwareInterface>hardware_interface/PositionJointInterface</hardwareInterface>
+            <mechanicalReduction>1</mechanicalReduction>
          </actuator>
       </transmission>
@@ -207,5 +215,6 @@
          <visual>
             <geometry>
-               <mesh filename="package://fennee_description/meshes/stl/foot.stl" scale="0.001 0.001 0.001" />
+               <mesh filename="package://fennee_description/meshes/stl/foot.stl"
+                  scale="0.001 0.001 0.001" />
             </geometry>
             <origin rpy="0 0.40010 0" xyz="0 -0.01 0.015" />
@@ -243,9 +252,10 @@
    </xacro:macro>
    <!-- Robot Body -->
-   <link name="base_link"/>
+   <link name="base_link" />
    <link name="base_inertia">
       <visual>
          <geometry>
-            <mesh filename="package://fennee_description/meshes/stl/mainbody.stl" scale="0.001 0.001 0.001" />
+            <mesh filename="package://fennee_description/meshes/stl/mainbody.stl"
+               scale="0.001 0.001 0.001" />
          </geometry>
          <material name="black" />
@@ -270,5 +280,6 @@
       <visual>
          <geometry>
-            <mesh filename="package://fennee_description/meshes/stl/backpart.stl" scale="0.001 0.001 0.001" />
+            <mesh filename="package://fennee_description/meshes/stl/backpart.stl"
+               scale="0.001 0.001 0.001" />
          </geometry>
          <origin rpy="0 0 3.1416" xyz="0.042 0.055 -0.0195" />
@@ -296,5 +307,6 @@
       <visual>
          <geometry>
-            <mesh filename="package://fennee_description/meshes/stl/frontpart.stl" scale="0.001 0.001 0.001" />
+            <mesh filename="package://fennee_description/meshes/stl/frontpart.stl"
+               scale="0.001 0.001 0.001" />
          </geometry>
          <origin rpy="0 0 3.1416" xyz="0.042 0.055 -0.0205" />
@@ -320,7 +332,19 @@
    </joint>
    <!-- create Legs -->
-   <xacro:gen_full_leg_joint pos="front_left" shiftx="${shiftx}" shifty="${shifty}" shift="${shift}" left="true" />
-   <xacro:gen_full_leg_joint pos="front_right" shiftx="${shiftx}" shifty="-${shifty}" shift="-${shift}" left="false" />
-   <xacro:gen_full_leg_joint pos="rear_left" shiftx="-${shiftx}" shifty="${shifty}" shift="${shift}" left="true" />
-   <xacro:gen_full_leg_joint pos="rear_right" shiftx="-${shiftx}" shifty="-${shifty}" shift="-${shift}" left="false" />
+   <xacro:gen_full_leg_joint pos="front_left" shiftx="${shiftx}" shifty="${shifty}" shift="${shift}"
+      left="true" />
+   <xacro:gen_full_leg_joint pos="front_right" shiftx="${shiftx}" shifty="-${shifty}"
+      shift="-${shift}" left="false" />
+   <xacro:gen_full_leg_joint pos="rear_left" shiftx="-${shiftx}" shifty="${shifty}" shift="${shift}"
+      left="true" />
+   <xacro:gen_full_leg_joint pos="rear_right" shiftx="-${shiftx}" shifty="-${shifty}"
+      shift="-${shift}" left="false" />
+   <!-- Camera  -->
+   <xacro:include filename="$(find depthai_descriptions)/urdf/include/depthai_macro.urdf.xacro" />
+   <!-- <xacro:arg name="camera_model" default="OAK-D" /> -->
+   <xacro:arg name="camera_model"  default="OAK-D-LITE" />
+   <xacro:depthai_camera camera_name="camera" parent="base_link"
+      camera_model="$(arg camera_model)" base_frame="oak-d_frame" cam_pos_x="${body_length + 0.004}"
+      cam_pos_y="0.0" cam_pos_z="-0.004" cam_roll="0.0"
+      cam_pitch="-0.174533" cam_yaw="0.0" />
 </robot>

Commit message: Fixing link for foxglove

File: fennee_description/urdf/fennee.urdf (robot description, URDF)
Before this commit: robot fennee, 32 links, 31 joints
Links:
- removed link camera_left_camera_frame
- removed link camera_left_camera_optical_frame
- removed link camera_model_origin
- removed link camera_rgb_camera_frame
- removed link camera_rgb_camera_optical_frame
- removed link camera_right_camera_frame
- removed link camera_right_camera_optical_frame
- added link _left_camera_frame
- added link _left_camera_optical_frame
- added link _model_origin; visual mesh filename=package://depthai_descriptions/urdf/models/OAK-D-LITE.stl
- added link _rgb_camera_frame
- added link _rgb_camera_optical_frame
- added link _right_camera_frame
- added link _right_camera_optical_frame
Joints:
- removed joint camera_center_joint
- removed joint camera_left_camera_joint
- removed joint camera_left_camera_optical_joint
- removed joint camera_model_origin_joint
- removed joint camera_rgb_camera_joint
- removed joint camera_rgb_camera_optical_joint
- removed joint camera_right_camera_joint
- removed joint camera_right_camera_optical_joint
- added joint _center_joint: type fixed, parent base_link, child oak-d_frame, origin xyz=0.169 0.0 -0.004 rpy=0.0 -0.174533 0.0
- added joint _left_camera_joint: type fixed, parent oak-d_frame, child _left_camera_frame, origin xyz=0 0.0375 0 rpy=0 0 0
- added joint _left_camera_optical_joint: type fixed, parent _left_camera_frame, child _left_camera_optical_frame, origin xyz=0 0 0 rpy=-1.5707963267948966 0.0 -1.5707963267948966
- added joint _model_origin_joint: type fixed, parent oak-d_frame, child _model_origin, origin xyz=0 0 0 rpy=1.5708 0 1.5708
- added joint _rgb_camera_joint: type fixed, parent oak-d_frame, child _rgb_camera_frame, origin xyz=0 0 0 rpy=0 0 0
- added joint _rgb_camera_optical_joint: type fixed, parent _rgb_camera_frame, child _rgb_camera_optical_frame, origin xyz=0 0 0 rpy=-1.5707963267948966 0.0 -1.5707963267948966
- added joint _right_camera_joint: type fixed, parent oak-d_frame, child _right_camera_frame, origin xyz=0 -0.0375 0 rpy=0 0 0
- added joint _right_camera_optical_joint: type fixed, parent _right_camera_frame, child _right_camera_optical_frame, origin xyz=0 0 0 rpy=-1.5707963267948966 0.0 -1.5707963267948966

File: fennee_description/urdf/fennee.xacro (robot description, xacro)
@@ -344,5 +344,5 @@
    <!-- <xacro:arg name="camera_model" default="OAK-D" /> -->
    <xacro:arg name="camera_model"  default="OAK-D-LITE" />
-   <xacro:depthai_camera camera_name="camera" parent="base_link"
+   <xacro:depthai_camera camera_name="" parent="base_link"
       camera_model="$(arg camera_model)" base_frame="oak-d_frame" cam_pos_x="${body_length + 0.004}"
       cam_pos_y="0.0" cam_pos_z="-0.004" cam_roll="0.0"

Commit message: Fixed camera orientation

File: fennee_description/urdf/fennee.urdf (robot description, URDF)
Before this commit: robot fennee, 32 links, 31 joints
Joints:
- joint _center_joint: origin xyz=0.169 0.0 -0.004 rpy=0.0 -0.174533 0.0 -> xyz=0.169 0.0 -0.004 rpy=0.0 -0.174533 3.14159

File: fennee_description/urdf/fennee.xacro (robot description, xacro)
@@ -347,4 +347,4 @@
       camera_model="$(arg camera_model)" base_frame="oak-d_frame" cam_pos_x="${body_length + 0.004}"
       cam_pos_y="0.0" cam_pos_z="-0.004" cam_roll="0.0"
-      cam_pitch="-0.174533" cam_yaw="0.0" />
+      cam_pitch="-0.174533" cam_yaw="3.14159" />
 </robot>

Commit message: reversed lidar

File: fennee_description/urdf/fennee.urdf (robot description, URDF)
Before this commit: robot fennee, 32 links, 31 joints
Joints:
- joint _center_joint: origin xyz=0.169 0.0 -0.004 rpy=0.0 -0.174533 3.14159 -> xyz=0.169 0.0 -0.004 rpy=0.0 -0.174533 0.0

File: fennee_description/urdf/fennee.xacro (robot description, xacro)
@@ -347,4 +347,4 @@
       camera_model="$(arg camera_model)" base_frame="oak-d_frame" cam_pos_x="${body_length + 0.004}"
       cam_pos_y="0.0" cam_pos_z="-0.004" cam_roll="0.0"
-      cam_pitch="-0.174533" cam_yaw="3.14159" />
+      cam_pitch="-0.174533" cam_yaw="0.0" />
 </robot>

Commit message: Fixing camera yaw again

File: fennee_description/urdf/fennee.urdf (robot description, URDF)
Before this commit: robot fennee, 32 links, 31 joints
Joints:
- joint _center_joint: origin xyz=0.169 0.0 -0.004 rpy=0.0 -0.174533 3.14159 -> xyz=0.169 0.0 -0.004 rpy=0.0 -0.174533 0.0

Commit message: Updated IMU from camera

File: fennee_description/urdf/fennee.urdf (robot description, URDF)
Before this commit: robot fennee, 32 links, 31 joints
Links:
- added link _imu_frame
- added link imu_link, mass 0.001
- link _model_origin: geometry visual mesh filename=package://depthai_descriptions/urdf/models/OAK-D.stl
- link base_inertia: mass 2.80 -> 3.4
Joints:
- added joint _imu_joint: type fixed, parent oak-d_frame, child _imu_frame, origin xyz=0.0 -0.015 -0.013662 rpy=0 1.5708 0
- added joint imu_joint: type fixed, parent base_link, child imu_link

File: fennee_description/urdf/fennee.xacro (robot description, xacro)
@@ -269,5 +269,5 @@
       </collision>
       <inertial>
-         <mass value="2.80" />
+         <mass value="3.4" />
          <inertia ixx="100" ixy="0" ixz="0" iyy="100" iyz="0" izz="100" />
       </inertial>
@@ -342,9 +342,32 @@
    <!-- Camera  -->
    <xacro:include filename="$(find depthai_descriptions)/urdf/include/depthai_macro.urdf.xacro" />
-   <!-- <xacro:arg name="camera_model" default="OAK-D" /> -->
-   <xacro:arg name="camera_model"  default="OAK-D-LITE" />
+   <xacro:arg name="camera_model" default="OAK-D" />
    <xacro:depthai_camera camera_name="" parent="base_link"
       camera_model="$(arg camera_model)" base_frame="oak-d_frame" cam_pos_x="${body_length + 0.004}"
       cam_pos_y="0.0" cam_pos_z="-0.004" cam_roll="0.0"
       cam_pitch="-0.174533" cam_yaw="0.0" />
+   <gazebo>
+      <plugin name="imu_controller" filename="libhector_gazebo_ros_imu.so">
+            <updateRate>50.0</updateRate>
+            <bodyName>imu_link</bodyName>
+            <topicName>imu/data</topicName>
+            <accelDrift>0.005 0.005 0.005</accelDrift>
+            <accelGaussianNoise>0.005 0.005 0.005</accelGaussianNoise>
+            <rateDrift>0.005 0.005 0.005 </rateDrift>
+            <rateGaussianNoise>0.005 0.005 0.005 </rateGaussianNoise>
+            <headingDrift>0.005</headingDrift>
+            <headingGaussianNoise>0.005</headingGaussianNoise>
+      </plugin>
+   </gazebo>
+   <link name="imu_link">
+      <inertial>
+            <mass value="0.001"/>
+            <origin xyz="0 0 0" rpy="0 0 0"/>
+            <inertia ixx="1e-09" ixy="0.0" ixz="0.0" iyy="1e-09" iyz="0.0" izz="1e-09"/>
+      </inertial>
+   </link>
+   <joint name="imu_joint" type="fixed">
+      <parent link="base_link" />
+      <child link="imu_link" />
+   </joint>
 </robot>

Commit message: Working on imu

File: fennee_description/urdf/fennee.urdf (robot description, URDF)
Before this commit: robot fennee, 34 links, 33 joints
Joints:
- joint imu_joint: origin (none) -> xyz=0.0 0.0 0.0 rpy=3.14159 3.14159 3.14159

Commit message: Finally got slam working

File: fennee_description/urdf/fennee.urdf (robot description, URDF)
Before this commit: robot fennee, 34 links, 33 joints
Joints:
- joint _imu_joint: origin xyz=0.0 -0.015 -0.013662 rpy=0 1.5708 0 -> xyz=0.0 -0.015 -0.013662 rpy=-1.5708 3.14159 1.5708
- joint imu_joint: origin xyz=0.0 0.0 0.0 rpy=3.14159 3.14159 3.14159 -> xyz=0.0 -0.015 -0.013662 rpy=0 0 -1.570795

File: fennee_description/urdf/fennee.xacro (robot description, xacro)
@@ -30,4 +30,12 @@
    <!-- <xacro:property name="shifty" value="0.0395" /> -->
    <xacro:property name="shifty" value="0.04285" />
+   <xacro:property name="has_imu" value="true" />
+   <xacro:property name="imu_offset_x" value="0.0" />
+   <xacro:property name="imu_offset_y" value="-0.15" />
+   <xacro:property name="imu_offset_z" value="-0.04" />
+   <xacro:property name="imu_r" value="0" />
+   <xacro:property name="imu_p" value="0" />
+   <xacro:property name="imu_y" value="-1.570795" />
+   <!-- <origin rpy="0 0 -1.570795" xyz="0.0 -0.15 -0.04"/> -->
    <!-- Macros -->
    <xacro:macro name="gen_shoulder" params="name left">
@@ -343,8 +351,10 @@
    <xacro:include filename="$(find depthai_descriptions)/urdf/include/depthai_macro.urdf.xacro" />
    <xacro:arg name="camera_model" default="OAK-D" />
+   <!-- <origin rpy="-1.5708 3.14159 1.5708" xyz="0.0 -0.015 -0.013662"/> -->
+   <!-- pitch: 3.14159-0.174533 -->
    <xacro:depthai_camera camera_name="" parent="base_link"
       camera_model="$(arg camera_model)" base_frame="oak-d_frame" cam_pos_x="${body_length + 0.004}"
-      cam_pos_y="0.0" cam_pos_z="-0.004" cam_roll="0.0"
-      cam_pitch="-0.174533" cam_yaw="0.0" />
+      cam_pos_y="0.0" cam_pos_z="-0.004" cam_roll="-1.5708"
+      cam_pitch="2.967057" cam_yaw="1.5708" />
    <gazebo>
       <plugin name="imu_controller" filename="libhector_gazebo_ros_imu.so">
@@ -370,4 +380,5 @@
       <parent link="base_link" />
       <child link="imu_link" />
+      <origin xyz="${imu_offset_x} ${imu_offset_y} ${imu_offset_z}" rpy="${imu_r} ${imu_p} ${imu_y}" />
    </joint>
 </robot>
