Commit message: Generated urdf

File: fennee_description/urdf/fennee.urdf (robot description, URDF)
Before this commit: robot fennee, 34 links, 33 joints
Joints:
- joint _imu_joint: origin xyz=0.0 -0.015 -0.013662 rpy=-1.5708 3.14159 1.5708 -> xyz=0.0 -0.015 -0.013662 rpy=0 1.5708 0
- joint imu_joint: origin xyz=0.0 -0.015 -0.013662 rpy=0 0 -1.570795 -> xyz=0.0 -0.15 -0.04 rpy=0 0 -1.570795

File: fennee_description/urdf/fennee.xacro (robot description, xacro)
@@ -353,8 +353,13 @@
    <!-- <origin rpy="-1.5708 3.14159 1.5708" xyz="0.0 -0.015 -0.013662"/> -->
    <!-- pitch: 3.14159-0.174533 -->
+   <!-- TODO: Fix these, since the IMU needs to be rotated to 1.5708 3.14159 1.5708 -->
+   <!-- <xacro:depthai_camera camera_name="" parent="base_link"
+      camera_model="$(arg camera_model)" base_frame="oak-d_frame" cam_pos_x="${body_length + 0.004}"
+      cam_pos_y="0.0" cam_pos_z="-0.004" cam_roll="-1.5708"
+      cam_pitch="2.967057" cam_yaw="1.5708" /> -->
    <xacro:depthai_camera camera_name="" parent="base_link"
       camera_model="$(arg camera_model)" base_frame="oak-d_frame" cam_pos_x="${body_length + 0.004}"
-      cam_pos_y="0.0" cam_pos_z="-0.004" cam_roll="-1.5708"
-      cam_pitch="2.967057" cam_yaw="1.5708" />
+      cam_pos_y="0.0" cam_pos_z="-0.004" cam_roll="0.0"
+      cam_pitch="-0.174533" cam_yaw="0.0" />
    <gazebo>
       <plugin name="imu_controller" filename="libhector_gazebo_ros_imu.so">
